Commit message: save commit

File: robot_specific_config/abb_irb2600_support/urdf/irb2600_20_165_macro.xacro (robot description, xacro)
@@ -7,5 +7,5 @@
       <collision name="collision">
         <geometry>
-          <mesh filename="package://abb_irb2600_support/meshes/irb2600/collision/base_link.stl" />
+          <mesh filename="package://abb_irb2600_support/meshes/irb2600_20_165/collision/base_link.stl" />
         </geometry>
         <xacro:material_abb_yellow />
@@ -13,5 +13,5 @@
       <visual name="visual">
         <geometry>
-          <mesh filename="package://abb_irb2600_support/meshes/irb2600/visual/base_link.stl" />
+          <mesh filename="package://abb_irb2600_support/meshes/irb2600_20_165/visual/base_link.stl" />
         </geometry>
         <xacro:material_abb_graphite_white/>
@@ -21,5 +21,5 @@
       <collision name="collision">
         <geometry>
-          <mesh filename="package://abb_irb2600_support/meshes/irb2600/collision/link_1.stl" />
+          <mesh filename="package://abb_irb2600_support/meshes/irb2600_20_165/collision/link_1.stl" />
         </geometry>
         <xacro:material_abb_yellow />
@@ -27,5 +27,5 @@
       <visual name="visual">
         <geometry>
-          <mesh filename="package://abb_irb2600_support/meshes/irb2600/visual/link_1.stl" />
+          <mesh filename="package://abb_irb2600_support/meshes/irb2600_20_165/visual/link_1.stl" />
         </geometry>
         <xacro:material_abb_graphite_white/>
